File: pcb/bakeneko40.kicad_pcb (KiCad board)
At the start: 2 copper layers, 116 parts, among them J1 JST SH 4-pin, J2 AVR-ISP-6, SW1 SW_Push, U1 ATmega32U4-AU, U2 SRV05-4, Y1 16MHz

Commit message: pcb routing
Parts:
- C1, C2, C3, C4, C5, C6, D1, D10, D11, D12, D13, D14, D15, D16, D17, D18, D19, D2, D20, D21, D22, D23, D24, D25, D26, D27, D28, D29, D3, D30, D31, D32, D33, D34, D35, D36, D37, D38, D39, D4, D40, D41, D42, D43, D44, D45, D46, D47, D48, D49, D5, D6, D7, D8, D9, F1, J1, R1, R2, R3, R4, SW1, U2, Y1: moved to B.Cu
- C7: footprint Diode_SMD:D_SOD-123 -> Capacitor_SMD:C_0805_2012Metric; moved to B.Cu
- U1: value ATmega32U4-AU -> ATmega32U2-MU; footprint Package_QFP:TQFP-44_10x10mm_P0.8mm -> Package_DFN_QFN:QFN-32-1EP_5x5mm_P0.5mm_EP3.1x3.1mm; moved to B.Cu
- moved D49 246.8 mm to (281.0, 114.3), turned to 90 degrees
- moved D1 224.5 mm to (33.3, 57.1), turned to 90 degrees
- moved MX27 213.9 mm to (265.9, 76.2)
- moved D40 195.4 mm to (281.0, 95.2), turned to 90 degrees
- moved D47 194.4 mm to (233.4, 114.3), turned to 90 degrees
- moved D48 188.8 mm to (259.6, 114.3), turned to 90 degrees
- moved MX40 180.4 mm to (273.1, 95.2)
- moved D37 180.4 mm to (219.1, 95.2), turned to 90 degrees
- moved D39 169.8 mm to (259.6, 95.2), turned to 90 degrees
- moved D2 166.3 mm to (52.4, 57.1), turned to 90 degrees
- moved MX1 164.1 mm to (25.4, 57.1)
- moved MX48 163.2 mm to (251.6, 114.3)
- moved MX49 158.2 mm to (273.1, 114.3)
- moved D15 156.3 mm to (35.7, 76.2), turned to 90 degrees
- moved MX4 154.8 mm to (82.5, 57.1)
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Connections:
- D1 pad 1: ROW0 -> ROW1
- D10 pad 1: ROW0 -> ROW2
- D11 pad 1: ROW0 -> ROW1
- D12 pad 1: ROW0 -> ROW2
- D13 pad 1: ROW0 -> ROW1
- D14 pad 1: ROW0 -> ROW2
- D15 pad 1: ROW1 -> ROW3
- D16 pad 1: ROW1 -> ROW4
- D17 pad 1: ROW1 -> ROW3
- D18 pad 1: ROW1 -> ROW4
- D19 pad 1: ROW1 -> ROW3
- D2 pad 1: ROW0 -> ROW2
- D20 pad 1: ROW1 -> ROW4
- D21 pad 1: ROW1 -> ROW3
- D22 pad 1: ROW1 -> ROW4
- D23 pad 1: ROW1 -> ROW3
- D24 pad 1: ROW1 -> ROW4
- D25 pad 1: ROW1 -> ROW3
- D26 pad 1: ROW1 -> ROW4
- D27 pad 1: ROW1 -> ROW3
- D28 pad 1: ROW2 -> ROW5
- D29 pad 1: ROW2 -> ROW6
- D3 pad 1: ROW0 -> ROW1
- D30 pad 1: ROW2 -> ROW5
- D31 pad 1: ROW2 -> ROW6
- D32 pad 1: ROW2 -> ROW5
- D33 pad 1: ROW2 -> ROW6
- D34 pad 1: ROW2 -> ROW5
- D35 pad 1: ROW2 -> ROW6
- D36 pad 1: ROW2 -> ROW5
- D37 pad 1: ROW2 -> ROW6
- D38 pad 1: ROW2 -> ROW5
- D39 pad 1: ROW2 -> ROW6
- D4 pad 1: ROW0 -> ROW2
- D40 pad 1: ROW2 -> ROW5
- D41 pad 1: ROW3 -> ROW7
- D42 pad 1: ROW3 -> ROW8
- D43 pad 1: ROW3 -> ROW7
- D44 pad 1: ROW3 -> ROW8
- D45 pad 1: ROW3 -> ROW7
- D46 pad 1: ROW3 -> ROW8
- D47 pad 1: ROW3 -> ROW7
- D48 pad 1: ROW3 -> ROW8
- D49 pad 1: ROW3 -> ROW7
- D5 pad 1: ROW0 -> ROW1
- D6 pad 1: ROW0 -> ROW2
- D7 pad 1: ROW0 -> ROW1
- D8 pad 1: ROW0 -> ROW2
- D9 pad 1: ROW0 -> ROW1
- J2 pad 5: RESET -> Net-(J2-Pad5)
- MX1 pad 1: COL0 -> COL1
- MX10 pad 1: COL9 -> COL5
- MX11 pad 1: COL10 -> COL6
- MX12 pad 1: COL11 -> COL6
- MX13 pad 1: COL12 -> COL7
- MX14 pad 1: COL13 -> COL7
- MX15 pad 1: COL0 -> COL1
- MX18 pad 1: COL3 -> COL2
- MX19 pad 1: COL4 -> COL3
- MX20 pad 1: COL5 -> COL3
- MX21 pad 1: COL6 -> COL4
- MX22 pad 1: COL7 -> COL4
- MX23 pad 1: COL8 -> COL5
- MX24 pad 1: COL9 -> COL5
- MX25 pad 1: COL10 -> COL6
- MX26 pad 1: COL11 -> COL6
- MX27 pad 1: COL12 -> COL7
- MX28 pad 1: COL0 -> COL1
- MX31 pad 1: COL3 -> COL2
- MX32 pad 1: COL4 -> COL3
- MX33 pad 1: COL5 -> COL3
- MX34 pad 1: COL6 -> COL4
- MX35 pad 1: COL7 -> COL4
- MX36 pad 1: COL8 -> COL5
- MX37 pad 1: COL9 -> COL5
- MX38 pad 1: COL10 -> COL6
- MX39 pad 1: COL11 -> COL6
- MX4 pad 1: COL3 -> COL2
- MX40 pad 1: COL12 -> COL7
- MX41 pad 1: COL0 -> COL1
- MX48 pad 1: COL7 -> COL6
- MX49 pad 1: COL8 -> COL7
- MX5 pad 1: COL4 -> COL3
- MX6 pad 1: COL5 -> COL3
- MX7 pad 1: COL6 -> COL4
- MX8 pad 1: COL7 -> COL4
- MX9 pad 1: COL8 -> COL5
- R4 pad 2: Net-(R4-Pad2) -> Net-(J2-Pad5)
- SW1 pad 2: Net-(R4-Pad2) -> Net-(J2-Pad5)
- U1 pad 1: ROW0 -> Net-(C6-Pad1)
- U1 pad 10: MOSI -> SCK
- U1 pad 11: MISO -> COL1
- U1 pad 12: Net-(U1-Pad12) -> COL2
- U1 pad 13: Net-(R4-Pad2) -> Net-(R1-Pad2)
- U1 pad 14: +5V -> COL3
- U1 pad 15: GND -> ROW6
- U1 pad 16: Net-(C7-Pad1) -> ROW2
- U1 pad 17: Net-(C6-Pad1) -> Net-(U1-Pad17)
- U1 pad 18: Net-(U1-Pad18) -> ROW1
- U1 pad 19: COL8 -> ROW3
- U1 pad 2: +5V -> Net-(C7-Pad1)
- U1 pad 20: COL9 -> ROW4
- U1 pad 21: COL10 -> Net-(U1-Pad21)
- U1 pad 22: COL11 -> ROW5
- U1 pad 23: GND -> COL4
- U1 pad 24: +5V -> Net-(J2-Pad5)
- U1 pad 25: COL12 -> COL5
- U1 pad 26: COL13 -> COL6
- U1 pad 27: Net-(U1-Pad27) -> Net-(C1-Pad1)
- U1 pad 28: COL0 -> GND
- U1 pad 29: COL1 -> Net-(R2-Pad1)
- U1 pad 3: Net-(R3-Pad1) -> GND
- U1 pad 30: COL2 -> Net-(R3-Pad1)
- U1 pad 31: COL3 -> +5V
- U1 pad 32: COL4 -> +5V
- U1 pad 33: Net-(R1-Pad2) -> GND
- U1 pad 4: Net-(R2-Pad1) -> +5V
- U1 pad 5: GND -> COL7
- U1 pad 6: Net-(C1-Pad1) -> ROW7
- U1 pad 7: +5V -> ROW8
- U1 pad 8: COL7 -> MOSI
- U1 pad 9: SCK -> MISO
Routing:
- net ROW1: track 0.00 -> 414.2 mm, vias 0 -> 2
- net ROW2: track 0.00 -> 326.9 mm, vias 0 -> 2
- net ROW3: track 0.00 -> 304.3 mm, vias 0 -> 2
- net ROW5: track 0.00 -> 293.0 mm, vias 0 -> 4
- net ROW4: track 0.00 -> 271.8 mm, vias 0 -> 5
- net ROW7: track 0.00 -> 270.0 mm, vias 0 -> 2
- net COL1: track 0.00 -> 264.8 mm, vias 0 -> 1
- net COL6: track 0.00 -> 249.7 mm, vias 0 -> 1
- net ROW6: track 0.00 -> 233.1 mm, vias 0 -> 2
- net COL7: track 0.00 -> 225.8 mm, vias 0 -> 1
- net ROW8: track 0.00 -> 221.3 mm, vias 0 -> 2
- net COL2: track 0.00 -> 206.5 mm, vias 0 -> 1
- net COL5: track 0.00 -> 196.9 mm, vias 0 -> 1
- net GND: track 0.00 -> 170.1 mm, vias 0 -> 4
- net COL4: track 0.00 -> 155.2 mm, vias 0 -> 1
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- added copper zone on B.Cu, net GND
Other:
- board outline added: 266.7 x 78.6 mm
- net class Default: trace_width 0.25 -> 0.254
- net class Power added: clearance 0.2, trace_width 0.29972, via_dia 0.8, via_drill 0.4
- rule trace_min: 0.2 -> 0.127

Commit message: finished pcb
Parts:
- MX44: footprint MX_Only:MXOnly-2.25U-NoLED -> MX_Only:MXOnly-2.25U-ReversedStabilizers-NoLED
- MX45: footprint MX_Only:MXOnly-2.75U-NoLED -> MX_Only:MXOnly-2.75U-ReversedStabilizers-NoLED
- moved C4 28.3 mm to (152.1, 117.2), turned to 0 degrees
- moved C5 26.2 mm to (151.6, 102.4), turned to 180 degrees
- moved C3 22.5 mm to (148.3, 115.9), turned to 0 degrees
- moved SW1 19.5 mm to (154.0, 84.9)
- moved C2 17.3 mm to (132.4, 119.9), turned to 180 degrees
- moved C7 3.24 mm to (142.1, 120.7), turned to 270 degrees
- moved J1 2.64 mm to (181.8, 101.6), turned to 0 degrees
- moved J2 2.38 mm to (96.5, 111.3)
- moved R2 2.38 mm to (158.0, 103.2)
- moved R3 2.38 mm to (158.0, 105.6)
- moved Y1 2.04 mm to (138.6, 120.6)
- moved C6 1.92 mm to (144.5, 120.7), turned to 270 degrees
- moved C1 0.79 mm to (146.1, 106.4)
- moved U2 0.15 mm to (166.0, 104.4), turned to 270 degrees
Routing:
- net GND: track 170.1 -> 269.9 mm, vias 4 -> 7
- net +5V: track 93.8 -> 177.7 mm
- net VBUS: track 16.5 -> 38.9 mm, vias 0 -> 2
- net Net-(J2-Pad5): track 64.0 -> 86.2 mm, vias 6 -> 5
- net MOSI: track 42.2 -> 52.1 mm
- net D+: track 19.6 -> 27.2 mm
- net D-: track 19.4 -> 26.7 mm
- net Net-(D44-Pad2): track 0.00 -> 6.82 mm
- net Net-(C7-Pad1): track 15.5 -> 19.5 mm
- net SCK: track 62.0 -> 65.7 mm
- net ROW6: track 233.1 -> 236.1 mm
- net Net-(C6-Pad1): track 22.7 -> 25.7 mm
- net COL3: track 152.3 -> 155.1 mm
- net COL1: track 264.8 -> 262.4 mm
- net Net-(R3-Pad1): track 27.3 -> 25.0 mm, vias 2 -> 0
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- added copper zone on B.Cu, net (none)
Other:
- board size 266.7 x 78.6 mm -> 266.7 x 76.2 mm

Commit message: pcb cut edits
Other:
- outline, holes or cut-outs redrawn
- net class Edge added: clearance 0.2, trace_width 0.127, via_dia 0.8, via_drill 0.4
Changed lines of the file:
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@@
   (general
     (thickness 1.6)
-    (drawings 11)
+    (drawings 31)
     (tracks 1044)
     (zones 0)
@@
     (38 B.Mask user)
     (39 F.Mask user)
-    (40 Dwgs.User user)
+    (40 Dwgs.User user hide)
     (41 Cmts.User user)
     (42 Eco1.User user)
@@
     (add_net SCK)
   )
+  (net_class Edge ""
+    (clearance 0.2)
+    (trace_width 0.127)
+    (via_dia 0.8)
+    (via_drill 0.4)
+    (uvia_dia 0.3)
+    (uvia_drill 0.1)
+  )
   (net_class Power ""
     (clearance 0.2)
@@
     )
   )
+  (gr_line (start 68.612899 123.799999) (end 230.065645 123.8) (layer Edge.Cuts) (width 0.1))
+  (gr_line (start 279.4 123.825) (end 238.312899 123.799999) (layer Edge.Cuts) (width 0.1))
+  (gr_line (start 19.05 123.825) (end 60.365645 123.8) (layer Edge.Cuts) (width 0.1))
+  (gr_line (start 55.294356 47.65) (end 131.847101 47.65) (layer Edge.Cuts) (width 0.1))
+  (gr_line (start 243.347101 47.65) (end 140.094356 47.65) (layer Edge.Cuts) (width 0.1))
+  (gr_line (start 280.19375 47.625) (end 251.594356 47.65) (layer Edge.Cuts) (width 0.1))
+  (gr_line (start 18.25625 47.625) (end 47.047101 47.65) (layer Edge.Cuts) (width 0.1))
+  (gr_arc (start 230.065645 122.3) (end 230.065645 123.8) (angle -62.5) (layer Edge.Cuts) (width 0.1))
+  (gr_arc (start 238.311856 122.3) (end 236.981822 122.993548) (angle -62.5) (layer Edge.Cuts) (width 0.1))
+  (gr_arc (start 234.18875 124.45) (end 236.981822 122.993548) (angle -124.9) (layer Edge.Cuts) (width 0.1))
+  (gr_arc (start 68.611856 122.3) (end 67.281822 122.993548) (angle -62.5) (layer Edge.Cuts) (width 0.1))
+  (gr_arc (start 60.365645 122.3) (end 60.365645 123.8) (angle -62.5) (layer Edge.Cuts) (width 0.1))
+  (gr_arc (start 64.48875 124.45) (end 67.281822 122.993548) (angle -124.9) (layer Edge.Cuts) (width 0.1))
+  (gr_arc (start 251.594356 49.15) (end 251.594356 47.65) (angle -62.5) (layer Edge.Cuts) (width 0.1))
+  (gr_arc (start 243.348145 49.15) (end 244.678179 48.456451) (angle -62.5) (layer Edge.Cuts) (width 0.1))
+  (gr_arc (start 247.47125 47) (end 244.678179 48.456451) (angle -124.9) (layer Edge.Cuts) (width 0.1))
+  (gr_arc (start 135.97125 47) (end 133.178179 48.456451) (angle -124.9) (layer Edge.Cuts) (width 0.1))
+  (gr_arc (start 131.848145 49.15) (end 133.178179 48.456451) (angle -62.5) (layer Edge.Cuts) (width 0.1))
+  (gr_arc (start 140.094356 49.15) (end 140.094356 47.65) (angle -62.5) (layer Edge.Cuts) (width 0.1))
+  (gr_arc (start 55.294356 49.15) (end 55.294356 47.65) (angle -62.5) (layer Edge.Cuts) (width 0.1))
+  (gr_arc (start 51.17125 47) (end 48.378179 48.456451) (angle -124.9) (layer Edge.Cuts) (width 0.1))
+  (gr_arc (start 47.048145 49.15) (end 48.378179 48.456451) (angle -62.5) (layer Edge.Cuts) (width 0.1))
   (dimension 58.375262 (width 0.15) (layer Dwgs.User)
     (gr_text "58.375 mm" (at 186.156244 76.816397 89.82823587) (layer Dwgs.User)
@@
   )
   (gr_line (start 15.875 50.00625) (end 15.875 120.65) (layer Edge.Cuts) (width 0.1))
-  (gr_line (start 19.05 123.825) (end 279.4 123.825) (layer Edge.Cuts) (width 0.1))
   (gr_arc (start 19.05 120.65) (end 15.875 120.65) (angle -90) (layer Edge.Cuts) (width 0.1))
   (gr_line (start 282.575 50.00625) (end 282.575 120.65) (layer Edge.Cuts) (width 0.1))
@@
     (arrow2b (pts (xy 15.875 85.725) (xy 17.001504 85.138579)))
   )
-  (gr_line (start 280.19375 47.625) (end 18.25625 47.625) (layer Edge.Cuts) (width 0.1))
   (gr_arc (start 280.19375 50.00625) (end 282.575 50.00625) (angle -90) (layer Edge.Cuts) (width 0.1))
   (gr_arc (start 18.25625 50.00625) (end 18.25625 47.625) (angle -90) (layer Edge.Cuts) (width 0.1))
-  (segment (start 166.05 105.92225) (end 166.05 105.3875) (width 0.29972) (layer B.Cu) (net 58) (status 30))
   (via (at 151.60625 100.0125) (size 0.8) (drill 0.4) (layers F.Cu B.Cu) (net 1))
   (segment (start 148.8875 100.0125) (end 146.50625 102.39375) (width 0.29972) (layer B.Cu) (net 1))
@@
   (segment (start 277.5575 109.22) (end 280.9875 112.65) (width 0.254) (layer B.Cu) (net 57) (status 20))
   (segment (start 275.59 109.22) (end 277.5575 109.22) (width 0.254) (layer B.Cu) (net 57) (status 10))
+  (segment (start 166.05 105.92225) (end 166.05 105.3875) (width 0.29972) (layer B.Cu) (net 58) (status 30))
   (segment (start 164.4625 100.9625) (end 164.30625 100.80625) (width 0.29972) (layer B.Cu) (net 58) (status 30))
   (segment (start 180.26875 106.375) (end 180.26875 107.06875) (width 0.29972) (layer B.Cu) (net 58) (status 30))
@@
   (segment (start 135.942309 112.852008) (end 135.288067 113.50625) (width 0.254) (layer B.Cu) (net 63))
   (segment (start 136.4383 112.852008) (end 135.942309 112.852008) (width 0.254) (layer B.Cu) (net 63) (status 10))
-  (segment (start 98.579462 110.33125) (end 98.168963 109.920751) (width 0.254) (layer B.Cu) (net 81))
-  (segment (start 96.427001 112.646749) (end 95.25 113.82375) (width 0.254) (layer B.Cu) (net 81) (status 20))
-  (segment (start 96.427001 110.741749) (end 96.427001 112.646749) (width 0.254) (layer B.Cu) (net 81))
-  (segment (start 97.247999 109.920751) (end 96.427001 110.741749) (width 0.254) (layer B.Cu) (net 81))
-  (segment (start 98.168963 109.920751) (end 97.247999 109.920751) (width 0.254) (layer B.Cu) (net 81))
+  (segment (start 92.86875 108.74375) (end 95.25 108.74375) (width 0.254) (layer B.Cu) (net 63) (status 20))
+  (segment (start 91.73526 107.61026) (end 92.86875 108.74375) (width 0.254) (layer B.Cu) (net 63))
+  (segment (start 91.73526 104.963056) (end 91.73526 107.61026) (width 0.254) (layer B.Cu) (net 63))
   (segment (start 21.59 71.27875) (end 23.97125 73.66) (width 0.254) (layer F.Cu) (net 64) (status 20))
   (segment (start 21.59 54.61) (end 21.59 71.27875) (width 0.254) (layer F.Cu) (net 64) (status 10))
@@
   (segment (start 148.2725 111.76) (end 143.618299 107.105799) (width 0.254) (layer B.Cu) (net 67))
   (segment (start 148.2725 111.76) (end 149.86 111.76) (width 0.254) (layer B.Cu) (net 67))
+  (segment (start 157.32125 111.76) (end 149.86 111.76) (width 0.254) (layer F.Cu) (net 67) (status 10))
+  (via (at 149.86 111.76) (size 0.8) (drill 0.4) (layers F.Cu B.Cu) (net 67))
   (segment (start 173.99 68.8975) (end 178.7525 73.66) (width 0.254) (layer F.Cu) (net 68) (status 20))
   (segment (start 173.99 54.61) (end 173.99 68.8975) (width 0.254) (layer F.Cu) (net 68) (status 10))
@@
   (segment (start 149.377346 117.627346) (end 150.01875 118.26875) (width 0.254) (layer B.Cu) (net 80))
   (segment (start 150.01875 118.26875) (end 153.9875 118.26875) (width 0.254) (layer B.Cu) (net 80))
+  (segment (start 98.579462 110.33125) (end 98.168963 109.920751) (width 0.254) (layer B.Cu) (net 81))
+  (segment (start 96.427001 112.646749) (end 95.25 113.82375) (width 0.254) (layer B.Cu) (net 81) (status 20))
+  (segment (start 96.427001 110.741749) (end 96.427001 112.646749) (width 0.254) (layer B.Cu) (net 81))
+  (segment (start 97.247999 109.920751) (end 96.427001 110.741749) (width 0.254) (layer B.Cu) (net 81))
+  (segment (start 98.168963 109.920751) (end 97.247999 109.920751) (width 0.254) (layer B.Cu) (net 81))
   (segment (start 138.90625 103.425) (end 137.55625 104.775) (width 0.254) (layer B.Cu) (net 81) (status 10))
   (segment (start 137.55625 104.775) (end 130.96875 104.775) (width 0.254) (layer B.Cu) (net 81))
@@
   (segment (start 142.08125 104.775) (end 140.73125 103.425) (width 0.254) (layer B.Cu) (net 81))
   (segment (start 103.1875 110.33125) (end 98.579462 110.33125) (width 0.254) (layer B.Cu) (net 81))
-  (segment (start 92.86875 108.74375) (end 95.25 108.74375) (width 0.254) (layer B.Cu) (net 63) (status 20))
-  (segment (start 91.73526 107.61026) (end 92.86875 108.74375) (width 0.254) (layer B.Cu) (net 63))
-  (segment (start 91.73526 104.963056) (end 91.73526 107.61026) (width 0.254) (layer B.Cu) (net 63))
-  (segment (start 157.32125 111.76) (end 149.86 111.76) (width 0.254) (layer F.Cu) (net 67) (status 10))
-  (via (at 149.86 111.76) (size 0.8) (drill 0.4) (layers F.Cu B.Cu) (net 67))
   (zone (net 1) (net_name GND) (layer B.Cu) (hatch edge 0.508)
     (connect_pads (clearance 0.02))
