File: pcb/bakeneko40.kicad_pcb (KiCad board)
At the start: 2 copper layers, 266.7 x 76.2 mm, 116 parts, among them J1 JST SH 4-pin, J2 AVR-ISP-6, SW1 SW_Push, U1 ATmega32U2-MU, U2 SRV05-4, Y1 16MHz

Commit message: final pcb and case
Parts:
- moved SW1 118.5 mm to (37.1, 65.7)
- moved C1 115.3 mm to (36.2, 71.4)
- moved R2 113.9 mm to (50.7, 64.8)
- moved R3 113.9 mm to (50.7, 67.1)
- moved U2 113.9 mm to (58.8, 66.0)
- moved C4 112.5 mm to (45.5, 80.9)
- moved J1 111.8 mm to (75.8, 66.0), turned to 270 degrees
- moved C5 111.1 mm to (45.0, 71.0), turned to 0 degrees
- moved F1 110.8 mm to (56.1, 71.2)
- moved R4 104.7 mm to (36.0, 83.5)
- moved C3 103.8 mm to (47.4, 91.7)
- moved C6 101.2 mm to (51.0, 81.8), turned to 0 degrees
- moved U1 99.7 mm to (42.2, 86.7), turned to 180 degrees
- moved C7 96.5 mm to (51.0, 88.5), turned to 0 degrees
- moved C2 96.2 mm to (45.5, 78.5), turned to 0 degrees
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Connections:
- U1 pad 10: SCK -> COL6
- U1 pad 11: COL1 -> COL5
- U1 pad 12: COL2 -> COL4
- U1 pad 15: ROW6 -> COL1
- U1 pad 16: ROW2 -> ROW8
- U1 pad 17: Net-(U1-Pad17) -> ROW7
- U1 pad 18: ROW1 -> ROW5
- U1 pad 19: ROW3 -> SCK
- U1 pad 20: ROW4 -> MOSI
- U1 pad 21: Net-(U1-Pad21) -> MISO
- U1 pad 22: ROW5 -> ROW2
- U1 pad 23: COL4 -> ROW1
- U1 pad 25: COL5 -> ROW3
- U1 pad 26: COL6 -> ROW4
- U1 pad 5: COL7 -> COL2
- U1 pad 6: ROW7 -> ROW6
- U1 pad 7: ROW8 -> Net-(U1-Pad7)
- U1 pad 8: MOSI -> Net-(U1-Pad8)
- U1 pad 9: MISO -> COL7
Routing:
- net ROW1: track 413.8 -> 285.2 mm, vias 2 -> 0
- net GND: track 269.9 -> 148.4 mm, vias 7 -> 4
- net COL4: track 156.1 -> 264.7 mm, vias 1 -> 0
- net COL5: track 197.3 -> 299.7 mm, vias 1 -> 0
- net COL7: track 225.2 -> 325.7 mm, vias 1 -> 0
- net COL6: track 249.9 -> 346.7 mm, vias 1 -> 0
- net +5V: track 177.7 -> 86.8 mm, vias 6 -> 5
- net COL1: track 262.4 -> 183.8 mm, vias 1 -> 0
- net COL3: track 155.1 -> 223.0 mm, vias 1 -> 0
- net SCK: track 65.7 -> 19.3 mm
- net MISO: track 61.4 -> 19.1 mm
- net ROW3: track 303.6 -> 263.4 mm
- net ROW4: track 269.8 -> 233.9 mm, vias 4 -> 2
- net MOSI: track 52.1 -> 16.2 mm
- net Net-(J2-Pad5): track 86.2 -> 53.3 mm, vias 5 -> 2
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- removed copper zone on B.Cu, net (none)
