File: pcb/qfp/bakeneko40.kicad_pcb (KiCad board)
At the start: 2 copper layers, 266.7 x 76.2 mm, 116 parts, among them J1 JST SH 4-pin, J2 AVR-ISP-6, SW1 SW_Push, U1 ATmega32U2-AU, U2 SRV05-4, Y1 16MHz

Commit message: pcb and qmk edits
Parts:
- moved R4 1.03 mm to (33.6, 80.5)
Connections:
- U1 pad 22: ROW2 -> ROW1
- U1 pad 23: ROW1 -> ROW2
Routing:
- net COL6: track 889.0 -> 482.1 mm
- net ROW2: track 315.2 -> 299.8 mm, vias 0 -> 2
- net ROW1: track 283.9 -> 277.2 mm, vias 0 -> 2
- net ROW5: track 287.6 -> 284.7 mm
- net Net-(J2-Pad5): track 56.5 -> 53.9 mm, vias 3 -> 2
- net COL5: track 296.8 -> 298.4 mm
- net GND: track 155.8 -> 154.3 mm
- net COL7: track 322.4 -> 323.9 mm
- net +5V: track 81.1 -> 81.8 mm
